Commit message: beacon sensor added

File: bluerov2_description/urdf/sensors.xacro (robot description, xacro)
@@ -17,4 +17,8 @@
     <origin xyz="0 0 0" rpy="0 0 0"/>
   </xacro:default_pressure>
+  <!-- Beacon Sensor  -->
+  <xacro:default_beacon namespace="${namespace}" parent_link="${namespace}/base_link">
+    <origin xyz="0 0 0" rpy="0 0 0"/>
+  </xacro:default_beacon>
   <!-- Mount a camera -->
   <!-- <xacro:default_camera namespace="${namespace}" parent_link="${namespace}/base_link" suffix="front">
