Commit message: Reconfiguring the trusters for Ros Melodic

File: bluerov2_description/urdf/gazebo.xacro (robot description, xacro)
@@ -1,31 +1,39 @@
 <?xml version="1.0"?>
+<!-- Copyright (c) 2016 The UUV Simulator Authors.
+     All rights reserved.
+     Licensed under the Apache License, Version 2.0 (the "License");
+     you may not use this file except in compliance with the License.
+     You may obtain a copy of the License at
+       http://www.apache.org/licenses/LICENSE-2.0
+     Unless required by applicable law or agreed to in writing, software
+     distributed under the License is distributed on an "AS IS" BASIS,
+     WITHOUT WARRANTIES OR CONDITIONS OF ANY KIND, either express or implied.
+     See the License for the specific language governing permissions and
+     limitations under the License.
+-->
 <robot xmlns:xacro="http://www.ros.org/wiki/xacro">
-  <xacro:macro name="bluerov2_hydro_model" params="namespace">
-    <!-- List of hydrodynamic models this robot's links -->
-    <link name="${namespace}/base_link">
-      <!-- This flag will make the link neutrally buoyant -->
-      <neutrally_buoyant>0</neutrally_buoyant>
-      <!-- Link's volume -->
-      <volume>${volume}</volume>
-      <!-- Link's bounding box, it is used to recalculate the immersed
-        volume when close to the surface.
-        This is a workaround the invalid bounding box given by Gazebo-->
-      <box>
-        <width>${x_size}</width>
-        <length>${y_size}</length>
-        <height>${z_size}</height>
-      </box>
-      <!-- Center of buoyancy -->
-      <center_of_buoyancy>${cob}</center_of_buoyancy>
-      <!-- Fossen's equation of motion for underwater vehicles
-      Reference:
-          [1] Fossen, Thor I. Handbook of marine craft hydrodynamics and motion
-          control. John Wiley & Sons, 2011.
-     -->
-      <hydrodynamic_model>
-          <type>fossen</type>
-          <!-- Added mass: see p.28 in Berg2012 -->
-          <added_mass>
-            1.7182 0 0 0 0 0
+    <!--
+    Center of buoyancy according to eq. (3.1) p. 28 in Berg2012.
+    The original values, [0.0822, -0.00773, 0.3872] however, seem to
+    assume NWU (otherwise cob is below cog?).
+    -->
+    <xacro:property name="cob" value="0.0 0.0 0.3"/>
+    <!-- Volume, see p.31 in Berg2012 -->
+    <xacro:property name="volume" value="0.011054"/>
+    <xacro:macro name="bluerov2_hydro_model" params="namespace">
+        <link name="${namespace}/base_link">
+            <neutrally_buoyant>0</neutrally_buoyant>
+            <volume>${volume}</volume>
+            <box>
+                <width>0.338</width>
+                <length>0.457</length>
+                <height>0.254</height>
+            </box>
+            <center_of_buoyancy>${cob}</center_of_buoyancy>
+            <hydrodynamic_model>
+                <type>fossen</type>
+                <!-- Added mass: see p.28 in Berg2012 -->
+                <added_mass>
+                      1.7182 0 0 0 0 0
             0 0 0 0 0 0
             0 0 5.468 0 0 0
@@ -33,51 +41,15 @@
             0 0 0 0 1.2481 0
             0 0 0 0 0 0.4006
-          </added_mass>
-          <!--
-            The linear damping coefficients can be provided as a diagonal (6 elements)
-            or a full matrix (36 coefficients), like the added-mass coefficients above
-            Linear damping: see p.31 in Berg2012
-          -->
-          <linear_damping>
-            -11.7391 -20 -31.8678 -25 -44.9085 -5
-          </linear_damping>
-          <!--
-            The linear damping coefficients proportional to the forward speed
-            can be provided as a diagonal (6 elements) or a full matrix (36 coefficients),
-            like the added-mass coefficients above.
-            This matrix is mostly useful for slender bodies (e.g. AUVs with torpedo shape)
-          -->
-          <!-- <linear_damping_forward_speed>
-            0 0 0 0 0 0
-          </linear_damping_forward_speed> -->
-          <!--
-            The quadratic damping coefficients can be provided as a diagonal (6 elements)
-            or a full matrix (36 coefficients), like the added-mass coefficients above
-            Non-linear damping: see p.30 in Berg2012
-          -->
-          <quadratic_damping>
-            0 0 0 0 0 0
-          </quadratic_damping>
-          <!--
-            In case you want to model a simple surface vessel, you can use the
-            implementation of linear (small angle) theory for boxed shaped vessels
-            by providing the following parameters. If you omit the area of the
-            water level plane area, it will be calculated from the bounding box
-            parameters. Uncomment the lines below in case you are simulating a
-            surface vessel.
-            For more details on these parameters and the computation of buoyancy
-            for vessels using this theory, check:
-              [1] Lecture Notes  TTK 4190 Guidance and Control of Vehicles (T. I. Fossen)
-                  http://www.fossen.biz/wiley/Ch4.pdf
-              [2] Fossen, Thor I. Handbook of marine craft hydrodynamics and motion
-                  control. John Wiley & Sons, 2011.
-          -->
-          <!--
-          <metacentric_width>0.0</metacentric_width>
-          <metacentric_length>0.0</metacentric_length>
-          <water_level_plane_area>0.0</water_level_plane_area>
-          -->
-      </hydrodynamic_model>
-    </link>
-  </xacro:macro>
+                </added_mass>
+                <!-- Linear damping: see p.31 in Berg2012 -->
+                <linear_damping>
+                    -11.7391 -20 -31.8678 -25 -44.9085 -5
+                </linear_damping>
+                <!-- Non-linear damping: see p.30 in Berg2012 -->
+                <quadratic_damping>
+                    0 0 0 0 0 0
+                </quadratic_damping>
+            </hydrodynamic_model>
+        </link>
+    </xacro:macro>
 </robot>

File: bluerov2_description/urdf/sensors.xacro (robot description, xacro)
@@ -23,5 +23,5 @@
   <!-- Mount a camera -->
   <xacro:default_camera namespace="${namespace}" parent_link="${namespace}/base_link" suffix="front">
-    <origin xyz="0 0 0.2" rpy="0 0 0"/>
+    <origin xyz="0 0 0.02" rpy="0 0 0"/>
   </xacro:default_camera>
 </robot>

File: bluerov2_description/urdf/snippets.xacro (robot description, xacro)
@@ -1,58 +1,27 @@
 <?xml version="1.0"?>
-<robot xmlns:xacro="http://www.ros.org/wiki/xacro">
-  <!-- MACRO FOR THRUSTER UNITS  -->
-  <!-- Provide the propeller mesh in a separate file with the rotation axis
-  over propeller's frame X-axis in DAE (Collada) or STL format.
-  -->
-  <xacro:property name="prop_mesh_file" value="file://$(find bluerov2_description)/meshes/bluerov2_propcw.dae"/>
-  <!--
-    Thruster macro with integration of joint and link. The thrusters should
-    be initialized in the actuators.xacro file.
-  -->
-  <xacro:macro name="thruster_macro" params="robot_namespace thruster_id *origin">
-    <!--
-    Dummy link as place holder for the thruster frame,
-    since thrusters can often be inside the collision geometry
-    of the vehicle and may cause internal collisions if set otherwise
-    -->
-    <link name="${robot_namespace}/thruster_${thruster_id}">
-      <visual>
-        <geometry>
-          <mesh filename="${prop_mesh_file}" scale="1 1 1" />
-        </geometry>
-      </visual>
-      <inertial>
-        <mass value="0.010" />
-        <origin xyz="0 0 0" rpy="0 0 0"/>
-        <inertia ixx="0.000000017" ixy="0.0" ixz="0.0"
-               iyy="0.000000017" iyz="0.0"
-               izz="0.000000017" />
-      </inertial>
-    </link>
-    <!-- Joint between thruster link and vehicle base link -->
-    <joint name="${robot_namespace}/thruster_${thruster_id}_joint" type="continuous">
-      <xacro:insert_block name="origin" />
-      <axis xyz="1 0 0" />
-      <parent link="${robot_namespace}/base_link" />
-      <child link="${robot_namespace}/thruster_${thruster_id}" />
-    </joint>
-    <!-- From desistek underwater vehicle -->
-    <gazebo>
-	    <!-- Thruster ROS plugin -->
-	    <xacro:macro name="thruster_macro"
+<!-- Copyright (c) 2016 The UUV Simulator Authors.
+     All rights reserved.
+     Licensed under the Apache License, Version 2.0 (the "License");
+     you may not use this file except in compliance with the License.
+     You may obtain a copy of the License at
+       http://www.apache.org/licenses/LICENSE-2.0
+     Unless required by applicable law or agreed to in writing, software
+     distributed under the License is distributed on an "AS IS" BASIS,
+     WITHOUT WARRANTIES OR CONDITIONS OF ANY KIND, either express or implied.
+     See the License for the specific language governing permissions and
+     limitations under the License.
+-->
+<robot xmlns:xacro="http://www.ros.org/wiki/xacro" >
+  <!-- Thruster joint and link snippet -->
+  <xacro:macro name="thruster_macro"
     params="robot_namespace thruster_id *origin">
     <xacro:thruster_module_first_order_basic_fcn_macro
       namespace="${robot_namespace}"
       thruster_id="${thruster_id}"
-      mesh_filename="${prop_mesh_file}"
+      mesh_filename="file://$(find bluerov2_description)/meshes/bluerov2_propcw.dae"
       dyn_time_constant="0.05"
-      rotor_constant="0.00001">
+      rotor_constant="0.01">
       <xacro:insert_block name="origin"/>
     </xacro:thruster_module_first_order_basic_fcn_macro>
   </xacro:macro>
-   </gazebo>
-    <gazebo reference="${robot_namespace}/thruster_${thruster_id}">
-      <selfCollide>false</selfCollide>
-    </gazebo>
-  </xacro:macro>
 </robot>
